File: 3.2.1 integrator_invertiertes/integrator.kicad_sch (KiCad schematic)
At the start: 7 parts, among them U1 TL072

Commit message: adding lagpass and allpass
Parts:
- R1: value 10k -> 1meg
Changed lines of the file:
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@@
     (pin "1")
     (instances
-      (project "TiefpassAktiv"
+      (project "3"
         (path "/b35302b3-1aa5-424e-90db-f5cc7fa728aa"
           (reference "V2") (unit 1)
@@
     (pin "1")
     (instances
-      (project "TiefpassAktiv"
+      (project "3"
         (path "/b35302b3-1aa5-424e-90db-f5cc7fa728aa"
           (reference "#PWR03") (unit 1)
@@
       (effects (font (size 1.27 1.27)))
     )
-    (property "Value" "10k" (at 53.34 20.32 90)
+    (property "Value" "1meg" (at 53.34 20.32 90)
       (effects (font (size 1.27 1.27)))
     )
@@
     (pin "1")
     (instances
-      (project "TiefpassAktiv"
+      (project "3"
         (path "/b35302b3-1aa5-424e-90db-f5cc7fa728aa"
           (reference "R1") (unit 1)
@@
     (pin "1")
     (instances
-      (project "TiefpassAktiv"
+      (project "3"
         (path "/b35302b3-1aa5-424e-90db-f5cc7fa728aa"
           (reference "V1") (unit 1)
@@
     (pin "1")
     (instances
-      (project "TiefpassAktiv"
+      (project "3"
         (path "/b35302b3-1aa5-424e-90db-f5cc7fa728aa"
           (reference "C1") (unit 1)
@@
     (pin "7")
     (instances
-      (project "TiefpassAktiv"
+      (project "3"
         (path "/b35302b3-1aa5-424e-90db-f5cc7fa728aa"
           (reference "U1") (unit 3)
@@
     (pin "7")
     (instances
-      (project "TiefpassAktiv"
+      (project "3"
         (path "/b35302b3-1aa5-424e-90db-f5cc7fa728aa"
           (reference "U1") (unit 1)
@@
     (pin "1")
     (instances
-      (project "TiefpassAktiv"
+      (project "3"
         (path "/b35302b3-1aa5-424e-90db-f5cc7fa728aa"
           (reference "#PWR05") (unit 1)
@@
     (pin "1")
     (instances
-      (project "TiefpassAktiv"
+      (project "3"
         (path "/b35302b3-1aa5-424e-90db-f5cc7fa728aa"
           (reference "R2") (unit 1)
@@
     (pin "1")
     (instances
-      (project "TiefpassAktiv"
+      (project "3"
         (path "/b35302b3-1aa5-424e-90db-f5cc7fa728aa"
           (reference "#PWR01") (unit 1)
@@
     (pin "1")
     (instances
-      (project "TiefpassAktiv"
+      (project "3"
         (path "/b35302b3-1aa5-424e-90db-f5cc7fa728aa"
           (reference "#PWR02") (unit 1)
@@
     (pin "7")
     (instances
-      (project "TiefpassAktiv"
+      (project "3"
         (path "/b35302b3-1aa5-424e-90db-f5cc7fa728aa"
           (reference "U1") (unit 2)
@@
     (pin "1")
     (instances
-      (project "TiefpassAktiv"
+      (project "3"
         (path "/b35302b3-1aa5-424e-90db-f5cc7fa728aa"
           (reference "#PWR06") (unit 1)
@@
     (pin "2")
     (instances
-      (project "TiefpassAktiv"
+      (project "3"
         (path "/b35302b3-1aa5-424e-90db-f5cc7fa728aa"
           (reference "V3") (unit 1)
@@
     (pin "1")
     (instances
-      (project "TiefpassAktiv"
+      (project "3"
         (path "/b35302b3-1aa5-424e-90db-f5cc7fa728aa"
           (reference "#PWR04") (unit 1)
