File: pifilter/pifilter.kicad_sch (KiCad schematic)
At the start: 8 parts, among them U1 TL072

Commit message: tiefpass3besselpluslagpass
Parts:
- removed Tl72: TL072, symbol Amplifier_Operational:TL072
- removed V4: VPULSE, symbol Simulation_SPICE:VPULSE
- added R3: 1meg, symbol Device:R
- added Tl1: TL072, symbol Amplifier_Operational:TL072
- added U2: ${SIM.PARAMS}, symbol Simulation_SPICE:OPAMP
- R1, R2: value 10 -> 10k
Connections:
- net Uein is gone; now on net 0: R1.1
- net 0: now also U2.1 (+), U2.4 (V-)
- net Ua: now also R3.2, U2.5
- net at C1.1, R2.2: now also R3.1
- net at U1.8 (V+), V3.1: now also U2.3 (V+)
- net at R1.2, R2.1: now also U2.2 (-)
