File: 4Te_Labor/4.1/hochpass_passive/hochpass_passive.kicad_sch (KiCad schematic)
At the start: 7 parts

Commit message: Update code plot
Other:
- note added: ".ac dec 10 1 1meg"
Changed lines of the file:
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@@
     (stroke (width 0) (type default))
+  )
+  (text ".ac dec 10 1 1meg" (at 76.835 47.625 0)
+    (effects (font (size 1.27 1.27)) (justify left bottom))
   )
   (global_label "U_e" (shape input) (at 93.98 30.48 90) (fields_autoplaced)
