File: 4Te_Labor/4.2/NE555_einstellbare_tastgrad/NE555_einstellbare_tastgrad.kicad_sch (KiCad schematic)
At the start: 9 parts, among them U1 NE555

Commit message: Update code plot
Parts:
- R2: value 3k -> 721
Changed lines of the file:
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@@
       (effects (font (size 1.27 1.27)))
     )
-    (property "Value" "3k" (at 134.62 73.66 90)
+    (property "Value" "721" (at 134.62 73.66 90)
       (effects (font (size 1.27 1.27)))
     )
