File: 4Te_Labor/4.2/NE555_monoflop/NE555_monoflop.kicad_sch (KiCad schematic)
At the start: 7 parts, among them U2 NE555

Commit message: Update code plot
Parts:
- R1: value 1k -> 721
Other:
- note added: ".tran 1u 1m"
- note removed: ".tran 100u 10m"
Changed lines of the file:
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@@
     (stroke (width 0) (type default))
   )
-  (text ".tran 100u 10m\n" (at 62.865 78.74 0)
+  (text ".tran 1u 1m\n" (at 62.865 78.74 0)
     (effects (font (size 1.27 1.27)) (justify left bottom))
   )
@@
       (effects (font (size 1.27 1.27)))
     )
-    (property "Value" "1k" (at 119.38 60.96 90)
+    (property "Value" "721" (at 119.38 60.96 90)
       (effects (font (size 1.27 1.27)))
     )
@@
       (effects (font (size 1.27 1.27)) (justify left) hide)
     )
-    (property "Sim.Params" "y1=0 y2=12 td=2n tr=2n tf=2n tw=0.99m per=1m" (at 12.7 66.04 0)
-      (effects (font (size 1.27 1.27)) (justify left))
-    )
+    (property "Sim.Params" "y1=0 y2=12 td=2n tr=2n tf=2n tw=145u per=150u" (at 12.7 66.04 0)
+      (effects (font (size 1.27 1.27)) (justify left))
+    )
