File: 4Te_Labor/4.2/NE555_oszcillator/NE555_oszcillator.kicad_sch (KiCad schematic)
At the start: 6 parts, among them U1 NE555

Commit message: Update code plot
Parts:
- R1: value 500 -> 721
- V1: value 12 -> 13
Connections:
- net U_tr: now reaches C1.2, R1.2, U1.2 (TR), U1.6 (THR)
Other:
- moved on the sheet: C2
Changed lines of the file:
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@@
+    (stroke (width 0) (type default))
+  )
+  (wire (pts (xy 113.665 71.755) (xy 114.935 71.755))
     (stroke (width 0) (type default))
   )
@@
     (stroke (width 0) (type default))
   )
-  (wire (pts (xy 102.235 71.755) (xy 107.315 71.755))
+  (wire (pts (xy 102.235 71.755) (xy 106.045 71.755))
     (stroke (width 0) (type default))
   )
@@
   (text ".tran 100n 1m\n" (at 87.63 90.805 0)
     (effects (font (size 1.27 1.27)) (justify left bottom))
+  )
+  (global_label "U_tr" (shape input) (at 153.67 64.77 0) (fields_autoplaced)
+    (effects (font (size 1.27 1.27)) (justify left))
+    (property "Intersheetrefs" "${INTERSHEET_REFS}" (at 160.4652 64.77 0)
+      (effects (font (size 1.27 1.27)) (justify left) hide)
+    )
   )
   (global_label "U_a" (shape input) (at 147.955 66.675 90) (fields_autoplaced)
@@
     )
   )
-  (symbol (lib_id "Device:C") (at 111.125 71.755 90) (unit 1)
-    (in_bom yes) (on_board yes) (dnp no) (fields_autoplaced)
-    (property "Reference" "C2" (at 111.125 64.135 90)
-      (effects (font (size 1.27 1.27)))
-    )
-    (property "Value" "100n" (at 111.125 66.675 90)
-      (effects (font (size 1.27 1.27)))
-    )
-    (property "Footprint" "" (at 114.935 70.7898 0)
-      (effects (font (size 1.27 1.27)) hide)
-    )
-    (property "Datasheet" "~" (at 111.125 71.755 0)
+  (symbol (lib_id "Device:C") (at 109.855 71.755 90) (unit 1)
+    (in_bom yes) (on_board yes) (dnp no) (fields_autoplaced)
+    (property "Reference" "C2" (at 109.855 64.135 90)
+      (effects (font (size 1.27 1.27)))
+    )
+    (property "Value" "100n" (at 109.855 66.675 90)
+      (effects (font (size 1.27 1.27)))
+    )
+    (property "Footprint" "" (at 113.665 70.7898 0)
+      (effects (font (size 1.27 1.27)) hide)
+    )
+    (property "Datasheet" "~" (at 109.855 71.755 0)
       (effects (font (size 1.27 1.27)) hide)
     )
@@
   (symbol (lib_id "Simulation_SPICE:VDC") (at 182.245 64.135 0) (unit 1)
     (in_bom yes) (on_board yes) (dnp no) (fields_autoplaced)
-    (property "Reference" "V1" (at 186.055 62.7352 0)
-      (effects (font (size 1.27 1.27)) (justify left))
-    )
-    (property "Value" "12" (at 186.055 65.2752 0)
+    (property "Reference" "V1" (at 186.69 62.7352 0)
+      (effects (font (size 1.27 1.27)) (justify left))
+    )
+    (property "Value" "13" (at 186.69 65.2752 0)
       (effects (font (size 1.27 1.27)) (justify left))
     )
@@
       (effects (font (size 1.27 1.27)) (justify left))
     )
-    (property "Value" "500" (at 150.495 74.295 0)
-      (effects (font (size 1.27 1.27)) (justify left))
-    )
+    (property "Value" "721" (at 150.495 74.295 0)
+      (effects (font (size 1.27 1.27)) (justify left))
+    )
