File: 4Te_Labor/4.3/DreieckRechteckoszillator/DreieckRechteckoszillator.kicad_sch (KiCad schematic)
At the start: 9 parts, among them U1 TL072

Commit message: Update the Plots
Parts:
- R1: value 2.7k -> 10k
- R3: value 10k -> 2.7k
- R4: value 10meg -> 1meg
Changed lines of the file:
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@@
       (effects (font (size 1.27 1.27)))
     )
-    (property "Value" "2.7k" (at 63.5 45.72 90)
+    (property "Value" "10k" (at 63.5 45.72 90)
       (effects (font (size 1.27 1.27)))
     )
@@
       (effects (font (size 1.27 1.27)))
     )
-    (property "Value" "10meg" (at 139.065 22.86 90)
+    (property "Value" "1meg" (at 139.065 22.86 90)
       (effects (font (size 1.27 1.27)))
     )
@@
       (effects (font (size 1.27 1.27)))
     )
-    (property "Value" "10k" (at 121.285 48.26 90)
+    (property "Value" "2.7k" (at 121.285 48.26 90)
       (effects (font (size 1.27 1.27)))
     )
