File: 5Te-Labor/5.3/test/test.kicad_sch (KiCad schematic)
At the start: 3 parts, among them U1 4081

Commit message: add phasendetector2
Connections:
- net GND: no longer U1.1
- net VCC: now also U1.1
Changed lines of the file:
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@@
 			)
 		)
-		(property "Sim.Library" "logic.lib"
+		(property "Sim.Library" "4081.dual.lib"
 			(at 346.71 99.06 0)
 			(effects
@@
 			)
 		)
-		(property "Sim.Name" "T_NAND"
+		(property "Sim.Name" "4081B"
 			(at 346.71 99.06 0)
 			(effects
@@
 			)
 		)
-		(property "Sim.Pins" "1=A 2=B 3=out 4=VCC 5=VSS"
+		(property "Sim.Pins" "1=A1 2=B1 3=Y1 4=Y2 5=A2 6=B2 7=VSS 8=A3 9=B3 10=Y3 11=Y4 12=A4 13=B4 14=VDD"
 			(at 346.71 99.06 0)
 			(effects
@@
 					(reference "U1")
 					(unit 4)
+				)
+			)
+		)
+	)
+	(symbol
+		(lib_id "power:VCC")
+		(at 52.07 66.04 0)
+		(unit 1)
+		(exclude_from_sim no)
+		(in_bom yes)
+		(on_board yes)
+		(dnp no)
+		(fields_autoplaced yes)
+		(property "Reference" "#PWR06"
+			(at 52.07 69.85 0)
+			(effects
+				(font
+					(size 1.27 1.27)
+				)
+				(hide yes)
+			)
+		)
+		(property "Value" "VCC"
+			(at 52.07 60.96 0)
+			(effects
+				(font
+					(size 1.27 1.27)
+				)
+			)
+		)
+		(property "Footprint" ""
+			(at 52.07 66.04 0)
+			(effects
+				(font
+					(size 1.27 1.27)
+				)
+				(hide yes)
+			)
+		)
+		(property "Datasheet" ""
+			(at 52.07 66.04 0)
+			(effects
+				(font
+					(size 1.27 1.27)
+				)
+				(hide yes)
+			)
+		)
+		(property "Description" ""
+			(at 52.07 66.04 0)
+			(effects
+				(font
+					(size 1.27 1.27)
+				)
+				(hide yes)
+			)
+		)
+		(pin "1"
+		)
+		(instances
+			(project "test"
+				(path "/e7dc5981-dedb-439b-b819-e1c0f358cf49"
+					(reference "#PWR06")
+					(unit 1)
 				)
 			)
@@
 			)
 		)
-		(property "Sim.Library" "logic.lib"
+		(property "Sim.Library" "4081.dual.lib"
 			(at 66.04 58.42 0)
 			(effects
@@
 			)
 		)
-		(property "Sim.Name" "T_NAND"
+		(property "Sim.Name" "4081B"
 			(at 66.04 58.42 0)
 			(effects
@@
 			)
 		)
-		(property "Sim.Pins" "1=A 2=B 3=out 4=VCC 5=VSS"
+		(property "Sim.Pins" "1=A1 2=B1 3=Y1 4=Y2 5=A2 6=B2 7=VSS 8=A3 9=B3 10=Y3 11=Y4 12=A4 13=B4 14=VDD"
 			(at 66.04 58.42 0)
 			(effects
@@
 	)
 	(symbol
-		(lib_id "power:GND")
-		(at 52.07 66.04 0)
-		(unit 1)
-		(exclude_from_sim no)
-		(in_bom yes)
-		(on_board yes)
-		(dnp no)
-		(fields_autoplaced yes)
-		(property "Reference" "#PWR06"
-			(at 52.07 72.39 0)
-			(effects
-				(font
-					(size 1.27 1.27)
-				)
-				(hide yes)
-			)
-		)
-		(property "Value" "GND"
-			(at 52.07 71.12 0)
-			(effects
-				(font
-					(size 1.27 1.27)
-				)
-			)
-		)
-		(property "Footprint" ""
-			(at 52.07 66.04 0)
-			(effects
-				(font
-					(size 1.27 1.27)
-				)
-				(hide yes)
-			)
-		)
-		(property "Datasheet" ""
-			(at 52.07 66.04 0)
-			(effects
-				(font
-					(size 1.27 1.27)
-				)
-				(hide yes)
-			)
-		)
-		(property "Description" ""
-			(at 52.07 66.04 0)
-			(effects
-				(font
-					(size 1.27 1.27)
-				)
-				(hide yes)
-			)
-		)
-		(pin "1"
-		)
-		(instances
-			(project "test"
-				(path "/e7dc5981-dedb-439b-b819-e1c0f358cf49"
-					(reference "#PWR06")
-					(unit 1)
-				)
-			)
-		)
-	)
-	(symbol
 		(lib_id "4xxx:4081")
 		(at 328.93 91.44 0)
@@
 			)
 		)
-		(property "Sim.Library" "logic.lib"
+		(property "Sim.Library" "4081.dual.lib"
 			(at 328.93 91.44 0)
 			(effects
@@
 			)
 		)
-		(property "Sim.Name" "T_NAND"
+		(property "Sim.Name" "4081B"
 			(at 328.93 91.44 0)
 			(effects
@@
 			)
 		)
-		(property "Sim.Pins" "1=A 2=B 3=out 4=VCC 5=VSS"
+		(property "Sim.Pins" "1=A1 2=B1 3=Y1 4=Y2 5=A2 6=B2 7=VSS 8=A3 9=B3 10=Y3 11=Y4 12=A4 13=B4 14=VDD"
 			(at 328.93 91.44 0)
 			(effects
@@
 			)
 		)
-		(property "Sim.Library" "logic.lib"
+		(property "Sim.Library" "4081.dual.lib"
 			(at 101.6 68.58 0)
 			(effects
@@
 			)
 		)
-		(property "Sim.Name" "T_NAND"
+		(property "Sim.Name" "4081B"
 			(at 101.6 68.58 0)
 			(effects
@@
 			)
 		)
-		(property "Sim.Pins" "1=A 2=B 3=out 4=VCC 5=VSS"
+		(property "Sim.Pins" "1=A1 2=B1 3=Y1 4=Y2 5=A2 6=B2 7=VSS 8=A3 9=B3 10=Y3 11=Y4 12=A4 13=B4 14=VDD"
 			(at 101.6 68.58 0)
 			(effects
@@
 			)
 		)
-		(property "Sim.Library" "logic.lib"
+		(property "Sim.Library" "4081.dual.lib"
 			(at 321.31 81.28 0)
 			(effects
@@
 			)
 		)
-		(property "Sim.Name" "T_NAND"
+		(property "Sim.Name" "4081B"
 			(at 321.31 81.28 0)
 			(effects
@@
 			)
 		)
-		(property "Sim.Pins" "1=A 2=B 3=out 4=VCC 5=VSS"
+		(property "Sim.Pins" "1=A1 2=B1 3=Y1 4=Y2 5=A2 6=B2 7=VSS 8=A3 9=B3 10=Y3 11=Y4 12=A4 13=B4 14=VDD"
 			(at 321.31 81.28 0)
 			(effects
