File: 5Te-Labor/5.3/phasendetector/phasendetector2.kicad_sch (KiCad schematic)
At the start: 11 parts, among them U1 4013, U2 4081, U3 4013, U4 TL072

Commit message: an attempt was made
Parts:
- removed U3: 4013, symbol 4xxx:4013
- added unit 2 of U1
- added unit 1 of U1
Connections:
- net GND: now also U1.6 (S), U1.8 (S)
- net U_REF: now also U1.3 (C)
- net U_REF2: now also U1.11 (C)
- net VCC: now also U1.5 (D), U1.9 (D)
- net qa: now reaches R1.1, U2.1
- net qa: now also U1.1 (Q)
- net reset: now reaches U2.3
- net reset: now also U1.10 (R), U1.4 (R)
- net qb: now reaches R2.1, U2.2
- net qb: now also U1.13 (Q)
- new net qabar: U1.2 (~{Q})
- new net qbbar: U1.12 (~{Q})
Other:
- note added: ".tran 1n 400n"
