File: 5Te-Labor/5.3/phasendetector/alleszussamen.kicad_sch (KiCad schematic)
At the start: 29 parts, among them Q1 BC337, Q2 BC327, U1 4013, U2 4081, U3 TL074, U4 TL072

Commit message: Update files
Other:
- note removed: ".tran 10u 10m"
Changed lines of the file:
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@@
-		)
-	)
-	(text ".tran 10u 10m\n"
-		(exclude_from_sim no)
-		(at 111.76 124.46 0)
-		(effects
-			(font
-				(size 1.27 1.27)
-			)
-			(justify right bottom)
 		)
 	)
