File: 5Te-Labor/5.3/test2/perfection.kicad_sch (KiCad schematic)
At the start: 7 parts, among them U1 4023, U2 4023, U3 4013

Commit message: an attempt was made
Parts:
- added U4, U5: 74AHC1G04, symbol 74xGxx:74AHC1G04
Connections:
- net GND: now also U4.3 (GND), U5.3 (GND)
- net VCC: now also U4.5 (VCC), U5.2, U5.5 (VCC); no longer U3.6 (S)
- net reset: now also U4.2; no longer U3.4 (R)
- new net: U3.4 (R), U4.4
- new net: U3.6 (S), U5.4
Other:
- moved on the sheet: V3
