File: 5Te-Labor/5.2/dreiecksrechteck-vco/dreiecksrechteck-vco.kicad_sch (KiCad schematic)
At the start: 11 parts, among them Q1 BC337, Q2 BC327, U1 TL072, U2 TL074

Commit message: Fuege schematic hinzu
Parts:
- added R5: 500, symbol Device:R
- added R6, R7: 1k, symbol Device:R
- added V1: 10, symbol Simulation_SPICE:VDC
Connections:
- net +12V: now also U2.4 (V+)
- net -12V: now also U2.11 (V-)
- net GND: now also U2.9 (-), V1.2
- net U_a: now also R1.1
- net U_o: now also R5.2
- net at U2.10 (+): now also R6.1, R7.1
- net at U2.8: now also Q2.1 (C), R6.2
- net at Q2.2 (B): now also Q1.2 (B), R5.1
- net at Q2.3 (E): now also Q1.3 (E), R3.1
- net U_c: now reaches U2.5 (+)
- net U_c: now also R7.2, V1.1
- net at U2.6 (-), U2.7: now also Q1.1 (C)
Other:
- moved on the sheet: R1, R2, R3, U2D

Commit message: quick save
Parts:
- removed U1: TL072, symbol Amplifier_Operational:TL072
Connections:
- net GND: now also U2.10 (+); no longer U2.9 (-)
- net at R6.1, R7.1: now also U2.9 (-); no longer U2.10 (+)
Changed lines of the file:
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@@
   (junction (at 124.46 77.47) (diameter 0) (color 0 0 0 0)
   )
-  (junction (at 227.33 102.87) (diameter 0) (color 0 0 0 0)
-  )
   (junction (at 106.68 90.17) (diameter 0) (color 0 0 0 0)
   )
@@
   (junction (at 64.77 69.85) (diameter 0) (color 0 0 0 0)
   )
-  (junction (at 227.33 81.28) (diameter 0) (color 0 0 0 0)
-  )
   (wire (pts (xy 34.29 101.6) (xy 43.18 101.6))
     (stroke (width 0) (type default))
@@
     (stroke (width 0) (type default))
   )
-  (wire (pts (xy 227.33 81.28) (xy 227.33 83.82))
-    (stroke (width 0) (type default))
-  )
   (wire (pts (xy 158.75 77.47) (xy 163.83 77.47))
     (stroke (width 0) (type default))
@@
   )
   (wire (pts (xy 227.33 62.23) (xy 227.33 71.12))
-    (stroke (width 0) (type default))
-  )
-  (wire (pts (xy 227.33 99.06) (xy 227.33 102.87))
     (stroke (width 0) (type default))
   )
@@
     )
   )
-  (symbol (lib_id "Amplifier_Operational:TL074") (at 48.26 116.84 0) (unit 3)
-    (in_bom yes) (on_board yes) (dnp no) (fields_autoplaced)
-    (property "Reference" "U2" (at 48.26 106.68 0)
-      (effects (font (size 1.27 1.27)))
-    )
-    (property "Value" "TL074" (at 48.26 109.22 0)
-      (effects (font (size 1.27 1.27)))
-    )
-    (property "Footprint" "" (at 46.99 114.3 0)
-      (effects (font (size 1.27 1.27)) hide)
-    )
-    (property "Datasheet" "http://www.ti.com/lit/ds/symlink/tl071.pdf" (at 49.53 111.76 0)
+  (symbol (lib_id "Amplifier_Operational:TL074") (at 48.26 116.84 0) (mirror x) (unit 3)
+    (in_bom yes) (on_board yes) (dnp no)
+    (property "Reference" "U2" (at 48.26 127 0)
+      (effects (font (size 1.27 1.27)))
+    )
+    (property "Value" "TL074" (at 48.26 124.46 0)
+      (effects (font (size 1.27 1.27)))
+    )
+    (property "Footprint" "" (at 46.99 119.38 0)
+      (effects (font (size 1.27 1.27)) hide)
+    )
+    (property "Datasheet" "http://www.ti.com/lit/ds/symlink/tl071.pdf" (at 49.53 121.92 0)
       (effects (font (size 1.27 1.27)) hide)
     )
@@
     )
   )
-  (symbol (lib_id "Amplifier_Operational:TL072") (at 229.87 91.44 0) (unit 3)
-    (in_bom yes) (on_board yes) (dnp no) (fields_autoplaced)
-    (property "Reference" "U1" (at 228.6 90.17 0)
-      (effects (font (size 1.27 1.27)) (justify left))
-    )
-    (property "Value" "TL072" (at 228.6 92.71 0)
-      (effects (font (size 1.27 1.27)) (justify left))
-    )
-    (property "Footprint" "" (at 229.87 91.44 0)
-      (effects (font (size 1.27 1.27)) hide)
-    )
-    (property "Datasheet" "http://www.ti.com/lit/ds/symlink/tl071.pdf" (at 229.87 91.44 0)
-      (effects (font (size 1.27 1.27)) hide)
-    )
-    (property "Sim.Library" "TL072-dual.lib" (at 229.87 91.44 0)
-      (effects (font (size 1.27 1.27)) hide)
-    )
-    (property "Sim.Name" "TL072c" (at 229.87 91.44 0)
-      (effects (font (size 1.27 1.27)) hide)
-    )
-    (property "Sim.Device" "SUBCKT" (at 229.87 91.44 0)
-      (effects (font (size 1.27 1.27)) hide)
-    )
-    (property "Sim.Pins" "1=1out 2=1in- 3=1in+ 4=vcc- 5=2in+ 6=2in- 7=2out 8=vcc+" (at 229.87 91.44 0)
-      (effects (font (size 1.27 1.27)) hide)
-    )
-    (pin "6")
-    (pin "4")
-    (pin "5")
-    (pin "1")
-    (pin "3")
-    (pin "2")
-    (pin "7")
-    (pin "8")
-    (instances
-      (project "dreiecksrechteck-vco"
-        (path "/2bfb4d56-aacb-4507-b57e-dbc901fa3ede"
-          (reference "U1") (unit 3)
-        )
-      )
-    )
-  )
   (symbol (lib_id "Device:R") (at 123.19 52.07 90) (unit 1)
     (in_bom yes) (on_board yes) (dnp no) (fields_autoplaced)
@@
     )
   )
-  (symbol (lib_id "Amplifier_Operational:TL072") (at 233.68 142.24 0) (mirror x) (unit 1)
-    (in_bom yes) (on_board yes) (dnp no)
-    (property "Reference" "U1" (at 233.68 151.765 0)
-      (effects (font (size 1.27 1.27)))
-    )
-    (property "Value" "TL072" (at 233.68 149.225 0)
-      (effects (font (size 1.27 1.27)))
-    )
-    (property "Footprint" "" (at 233.68 142.24 0)
-      (effects (font (size 1.27 1.27)) hide)
-    )
-    (property "Datasheet" "http://www.ti.com/lit/ds/symlink/tl071.pdf" (at 233.68 142.24 0)
-      (effects (font (size 1.27 1.27)) hide)
-    )
-    (property "Sim.Library" "TL072-dual.lib" (at 233.68 142.24 0)
-      (effects (font (size 1.27 1.27)) hide)
-    )
-    (property "Sim.Name" "TL072c" (at 233.68 142.24 0)
-      (effects (font (size 1.27 1.27)) hide)
-    )
-    (property "Sim.Device" "SUBCKT" (at 233.68 142.24 0)
-      (effects (font (size 1.27 1.27)) hide)
-    )
-    (property "Sim.Pins" "1=1out 2=1in- 3=1in+ 4=vcc- 5=2in+ 6=2in- 7=2out 8=vcc+" (at 233.68 142.24 0)
-      (effects (font (size 1.27 1.27)) hide)
-    )
-    (pin "6")
-    (pin "4")
-    (pin "5")
-    (pin "1")
-    (pin "3")
-    (pin "2")
-    (pin "7")
-    (pin "8")
-    (instances
-      (project "dreiecksrechteck-vco"
-        (path "/2bfb4d56-aacb-4507-b57e-dbc901fa3ede"
-          (reference "U1") (unit 1)
-        )
-      )
-    )
-  )
   (symbol (lib_id "Simulation_SPICE:VDC") (at 21.59 80.01 0) (unit 1)
     (in_bom yes) (on_board yes) (dnp no) (fields_autoplaced)
@@
         )
       )
-    )
-  )
-  (symbol (lib_id "Amplifier_Operational:TL072") (at 261.62 140.97 0) (unit 2)
-    (in_bom yes) (on_board yes) (dnp no) (fields_autoplaced)
-    (property "Reference" "U1" (at 261.62 131.445 0)
-      (effects (font (size 1.27 1.27)))
-    )
-    (property "Value" "TL072" (at 261.62 133.985 0)
-      (effects (font (size 1.27 1.27)))
-    )
-    (property "Footprint" "" (at 261.62 140.97 0)
-      (effects (font (size 1.27 1.27)) hide)
-    )
-    (property "Datasheet" "http://www.ti.com/lit/ds/symlink/tl071.pdf" (at 261.62 140.97 0)
-      (effects (font (size 1.27 1.27)) hide)
-    )
-    (property "Sim.Library" "TL072-dual.lib" (at 261.62 140.97 0)
-      (effects (font (size 1.27 1.27)) hide)
-    )
-    (property "Sim.Name" "TL072c" (at 261.62 140.97 0)
-      (effects (font (size 1.27 1.27)) hide)
-    )
-    (property "Sim.Device" "SUBCKT" (at 261.62 140.97 0)
-      (effects (font (size 1.27 1.27)) hide)
-    )
-    (property "Sim.Pins" "1=1out 2=1in- 3=1in+ 4=vcc- 5=2in+ 6=2in- 7=2out 8=vcc+" (at 261.62 140.97 0)
-      (effects (font (size 1.27 1.27)) hide)
-    )
-    (pin "6")
-    (pin "4")
-    (pin "5")
-    (pin "1")
-    (pin "3")
-    (pin "2")
-    (pin "7")
-    (pin "8")
-    (instances
-      (project "dreiecksrechteck-vco"
-        (path "/2bfb4d56-aacb-4507-b57e-dbc901fa3ede"
-          (reference "U1") (unit 2)
-        )
-      )

Commit message: Creating pdfs
Parts:
- V1: value 10 -> 3
