File: 5Te-Labor/5.2/experiment/vco.kicad_sch (KiCad schematic)
At the start: 15 parts, among them Q1 BC337, Q2 BC327, U2 TL074

Commit message: Update files
Parts:
- removed Q1: BC337, Package_TO_SOT_THT:TO-92_Inline, symbol Transistor_BJT:BC337
- removed Q2: BC327, Package_TO_SOT_THT:TO-92_Inline, symbol Transistor_BJT:BC327
- removed V1: 10, symbol Simulation_SPICE:VDC
- removed V4: VSIN, symbol Simulation_SPICE:VSIN
- added Q1: BC327, Package_TO_SOT_THT:TO-92_Inline, symbol Transistor_BJT:BC327
- added Q2: BC337, Package_TO_SOT_THT:TO-92_Inline, symbol Transistor_BJT:BC337
- R1: value 20k -> 1k
- R2: value 30k -> 1k
- R6: value 1k -> 20k
- R7: value 1k -> 30k
Connections:
- net U_o: now also R7.2; no longer R2.2
- net at U2.8: now also R2.2, Q1.1 (C); no longer R6.2
- net at R5.1: now also Q1.2 (B), Q2.2 (B)
- net at R3.1: now also Q1.3 (E), Q2.3 (E)
- net at U2.6 (-), U2.7: now also Q2.1 (C)
- net U_a: no longer names the net of C1.2, R4.2, U2.1
- net U_a: now also R6.1; no longer R1.1
- net U_c renamed U_ein
- net U_ein: now also R1.2; no longer R7.2
- new net: R1.1, R2.1, U2.9 (-)
- new net: R6.2, R7.1, U2.12 (+)
Other:
- removed sheet pifilter
