File: 5Te-Labor/5.3/allezussamen/alleszussamen.kicad_sch (KiCad schematic)
At the start: 29 parts, among them Q1 BC337, Q2 BC327, U1 4013, U2 4081, U3 TL074, U4 TL072

Commit message: pdf hinzufugen
Parts:
- added C3, C4: 1p, symbol Device:C
- added R16: 52, symbol Device:R
- added R17: 1k, symbol Device:R
Connections:
- net GND: now also R17.2
- net U_REF2: now also C4.2
- net U_c: now also C3.2
- net U_einvco: now reaches C1.2, D1.2 (A), U4.1
- net U_einvco: now also R16.2
- net U_o renamed U_outvco
- new net: C3.1, R16.1
- new net: C4.1, R17.1
Other:
- note added: ".option reltol=1 abstol=100meg chgtol=1"
- note added: ".tran 1u 4m"
- note removed: ".tran 1n 4u"

Commit message: Update files
Parts:
- removed C3, C4: 1p, symbol Device:C
- removed D1, D2: 1N5819, Diode_THT:D_DO-41_SOD81_P10.16mm_Horizontal, symbol Diode:1N5819
- removed R14: 1500, symbol Device:R
- removed R15: 100k, symbol Device:R
- removed R16: 52, symbol Device:R
- removed R17: 1k, symbol Device:R
Connections:
- net U_einvco is gone; now on net U_c: C1.2, U4.1
- net U_outvco is gone; now on net U_REF2: R11.2, R13.2, U3.14
Other:
- note added: ".tran 1n 4u"
- note removed: ".option reltol=1 abstol=100meg chgtol=1"
- note removed: ".tran 1u 4m"
